Commit message: update ros2 control file

File: epmc_sample_bot_description/urdf/ros2_control.xacro (robot description, xacro)
@@ -1,9 +1,9 @@
 <?xml version="1.0"?>
 <robot xmlns:xacro="http://www.ros.org/wiki/xacro">
-    <ros2_control name="epmc_hardware_interface" type="system">
+    <xacro:macro name="epmc_hardware_interface" params="name">
+    <ros2_control name="${name}_front" type="system">
       <hardware>
         <plugin>epmc_hardware_interface/EPMC_HardwareInterface</plugin>
-        <param name="supported_num_of_motors">4</param>
-        <param name="serial_port">/dev/ttyUSB0</param>
+        <param name="serial_port">/dev/ttyACM0</param>
         <param name="serial_baud_rate">115200</param>
         <param name="serial_timeout_ms">18</param>
@@ -11,6 +11,5 @@
         <param name="motor0_wheel_name">front_left_wheel_joint</param>
         <param name="motor1_wheel_name">front_right_wheel_joint</param>
-        <param name="motor2_wheel_name">rear_left_wheel_joint</param>
-        <param name="motor3_wheel_name">rear_right_wheel_joint</param>
+        <param name="cmd_vel_timeout_ms">2000</param>
       </hardware>
       <joint name="front_left_wheel_joint">
@@ -30,4 +29,15 @@
         <state_interface name="velocity"/>
       </joint>
+    </ros2_control>
+    <ros2_control name="${name}_rear" type="system">
+      <hardware>
+        <plugin>epmc_hardware_interface/EPMC_HardwareInterface</plugin>
+        <param name="serial_port">/dev/ttyACM1</param>
+        <param name="serial_baud_rate">115200</param>
+        <param name="serial_timeout_ms">18</param>
+        <param name="cmd_vel_timeout_ms">2000</param>
+        <param name="motor0_wheel_name">rear_left_wheel_joint</param>
+        <param name="motor1_wheel_name">rear_right_wheel_joint</param>
+      </hardware>
       <joint name="rear_left_wheel_joint">
         <command_interface name="velocity">
@@ -47,3 +57,5 @@
       </joint>
     </ros2_control>
+  </xacro:macro>
+  <xacro:epmc_hardware_interface name="epmc_hardware_interface"/>
 </robot>

Commit message: update ros2 control file

File: epmc_sample_bot_description/urdf/ros2_control.xacro (robot description, xacro)
@@ -1,9 +1,9 @@
 <?xml version="1.0"?>
 <robot xmlns:xacro="http://www.ros.org/wiki/xacro">
-    <xacro:macro name="epmc_hardware_interface" params="name">
-    <ros2_control name="${name}_front" type="system">
+    <ros2_control name="epmc_hardware_interface" type="system">
       <hardware>
         <plugin>epmc_hardware_interface/EPMC_HardwareInterface</plugin>
-        <param name="serial_port">/dev/ttyACM0</param>
+        <param name="supported_num_of_motors">4</param>
+        <param name="serial_port">/dev/ttyUSB0</param>
         <param name="serial_baud_rate">115200</param>
         <param name="serial_timeout_ms">18</param>
@@ -11,5 +11,6 @@
         <param name="motor0_wheel_name">front_left_wheel_joint</param>
         <param name="motor1_wheel_name">front_right_wheel_joint</param>
-        <param name="cmd_vel_timeout_ms">2000</param>
+        <param name="motor2_wheel_name">rear_left_wheel_joint</param>
+        <param name="motor3_wheel_name">rear_right_wheel_joint</param>
       </hardware>
       <joint name="front_left_wheel_joint">
@@ -29,15 +30,4 @@
         <state_interface name="velocity"/>
       </joint>
-    </ros2_control>
-    <ros2_control name="${name}_rear" type="system">
-      <hardware>
-        <plugin>epmc_hardware_interface/EPMC_HardwareInterface</plugin>
-        <param name="serial_port">/dev/ttyACM1</param>
-        <param name="serial_baud_rate">115200</param>
-        <param name="serial_timeout_ms">18</param>
-        <param name="cmd_vel_timeout_ms">2000</param>
-        <param name="motor0_wheel_name">rear_left_wheel_joint</param>
-        <param name="motor1_wheel_name">rear_right_wheel_joint</param>
-      </hardware>
       <joint name="rear_left_wheel_joint">
         <command_interface name="velocity">
@@ -57,5 +47,3 @@
       </joint>
     </ros2_control>
-  </xacro:macro>
-  <xacro:epmc_hardware_interface name="epmc_hardware_interface"/>
 </robot>
